File: M-N-SRAM-V8.brd (EAGLE design)
At the start: 100 x 70 mm, 38 parts, among them IC1 IS61WV20488BLL-10T, J1 CON-DSUB-15-VGA, Q1 BC546A

Commit message: Schematic Correction
Connections:
- removed net +33_3: JP2.11, X2.5, X3.5
- net +3.3V: now also JP1.29, X2.5, X3.5; no longer JP1.11
Routing:
- net +3.3V: track 39.7 -> 126.2 mm
- net +33_3: track 74.6 -> 0.00 mm
Changed lines of the file:
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@@
 <contactref element="IC1" pad="33"/>
 <contactref element="C1" pad="1"/>
-<contactref element="JP1" pad="11"/>
 <polygon width="0.1524" layer="1">
 <vertex x="64.77" y="11.43"/>
-<vertex x="64.77" y="6.35"/>
-<vertex x="65.4" y="5.08"/>
-<vertex x="65.4" y="3.4"/>
-<vertex x="63.5" y="3.4"/>
-<vertex x="63.5" y="6.35"/>
-<vertex x="59.69" y="10.16"/>
+<vertex x="64.77" y="8.89"/>
+<vertex x="62.23" y="8.89"/>
 <vertex x="59.69" y="11.43"/>
 </polygon>
@@
 <wire x1="64.77" y1="26.67" x2="63.373" y2="25.273" width="0.1524" layer="16"/>
 <wire x1="63.373" y1="25.273" x2="63.373" y2="10.16" width="0.1524" layer="16"/>
+<contactref element="JP1" pad="29"/>
+<polygon width="0.1524" layer="1">
+<vertex x="35.56" y="12.7"/>
+<vertex x="34.29" y="12.7"/>
+<vertex x="34.29" y="12"/>
+<vertex x="36.83" y="12"/>
+<vertex x="36.83" y="12.7"/>
+</polygon>
+<polygon width="0.1524" layer="1">
+<vertex x="43.18" y="5.08"/>
+<vertex x="43.18" y="0"/>
+<vertex x="33.02" y="0"/>
+<vertex x="33.02" y="12.7"/>
+<vertex x="36.83" y="12.7"/>
+<vertex x="36.83" y="5.08"/>
+</polygon>
+<contactref element="X2" pad="5"/>
+<contactref element="X3" pad="5"/>
+<wire x1="13.97" y1="21.9964" x2="9.2964" y2="21.9964" width="0.1524" layer="1"/>
+<wire x1="7.62" y1="20.32" x2="7.62" y2="8.89" width="0.1524" layer="1"/>
+<wire x1="7.62" y1="8.89" x2="8.89" y2="7.62" width="0.1524" layer="1"/>
+<wire x1="8.89" y1="7.62" x2="33.02" y2="7.62" width="0.1524" layer="1"/>
+<wire x1="9.2964" y1="21.9964" x2="7.62" y2="20.32" width="0.1524" layer="1"/>
+<wire x1="13.97" y1="57.5564" x2="9.2964" y2="57.5564" width="0.1524" layer="1"/>
+<wire x1="9.2964" y1="57.5564" x2="7.62" y2="55.88" width="0.1524" layer="1"/>
+<wire x1="7.62" y1="22.86" x2="7.62" y2="55.88" width="0.1524" layer="1"/>
+<wire x1="9.2964" y1="21.9964" x2="8.4836" y2="21.9964" width="0.1524" layer="1"/>
+<wire x1="8.4836" y1="21.9964" x2="7.62" y2="22.86" width="0.1524" layer="1"/>
 </signal>
 <signal name="BT_RST">
@@
 <wire x1="68.7194" y1="4.630325" x2="68.7194" y2="3.2294" width="0.1524" layer="16"/>
 </signal>
-<signal name="+33_3">
-<contactref element="JP2" pad="11"/>
-<contactref element="X3" pad="5"/>
-<contactref element="X2" pad="5"/>
-<wire x1="13.97" y1="57.5564" x2="37.2364" y2="57.5564" width="0.1524" layer="1"/>
-<wire x1="41.77" y1="62.09" x2="41.77" y2="64.53" width="0.1524" layer="1"/>
-<wire x1="37.2364" y1="57.5564" x2="41.77" y2="62.09" width="0.1524" layer="1"/>
-<wire x1="13.97" y1="21.9964" x2="16.9164" y2="21.9964" width="0.1524" layer="16"/>
-<wire x1="16.9164" y1="21.9964" x2="17.78" y2="22.86" width="0.1524" layer="16"/>
-<wire x1="17.78" y1="22.86" x2="17.78" y2="57.15" width="0.1524" layer="16"/>
-<wire x1="17.78" y1="57.15" x2="17.3736" y2="57.5564" width="0.1524" layer="16"/>
-<wire x1="17.3736" y1="57.5564" x2="13.97" y2="57.5564" width="0.1524" layer="16"/>
-</signal>
 </signals>
